File: hardware/pcb/v1/kaelix.kicad_pcb (KiCad board)
At the start: 2 copper layers, 42 x 42 mm, 35 parts, among them J1 LiPo 3,7V, J2 UART/BOOT, Q1 SI2301CDS, Q2 BC847B, Q3 SI2301CDS, U1 ESP32-S3-WROOM-1U-N16R8, U2 MPU-6050, U3 Ai-Thinker Ra-02 (SX1278), U4 HT7333

Commit message: fix(router): não conta plano sob o corpo de peça de passo fino
A grade do roteador via células de plano de terra na faixa entre as
fileiras de pads de um QFN de 0,5 mm e tratava a região como caminho. O
preenchimento do KiCad, com espessura mínima e folga exatas, deixa ali só
retalhos, e o escape seguinte ou uma pista de sinal os fecha em ilha. Na
v3 o escape de GND do U2.1 terminou numa dessas ilhas sob o MPU6050: o
roteador deu o pad por ligado e o DRC acusou um grupo de terra solto.

Agora, sob o corpo de peça de passo fino e na face dela, o plano não conta
como caminho. Atravessar com pista continua possível; só deixa de valer
contar com plano ali. A regra fica no modelo do plano (_gnd_ok), e não em
cada ponto de chegada, porque o escape inicial e a verificação final de
terra usam o mesmo modelo.

O roteamento da v1 e da v2 muda — costura 92 -> 71 e 261 -> 234, porque a
região deixou de oferecer plano dos dois lados — sem tocar em circuito nem
em placement. As duas seguem com ERC e DRC limpos e zero itens soltos.
Routing:
- net GND: track 6.74 -> 16.3 mm, vias 95 -> 74
Changed lines of the file:
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@@
 	)
 	(segment
+(start 148.1000 92.6000)
+(end 146.9000 91.4000)
+(width 0.2)
+(layer "B.Cu")
+(net 4)
+	)
+	(segment
+(start 146.9000 91.4000)
+(end 145.4000 91.4000)
+(width 0.2)
+(layer "B.Cu")
+(net 4)
+	)
+	(segment
+(start 145.4000 91.4000)
+(end 145.3000 91.3000)
+(width 0.2)
+(layer "B.Cu")
+(net 4)
+	)
+	(segment
+(start 145.3000 91.3000)
+(end 144.6000 91.3000)
+(width 0.2)
+(layer "B.Cu")
+(net 4)
+	)
+	(segment
+(start 144.6000 91.3000)
+(end 143.0000 89.7000)
+(width 0.2)
+(layer "B.Cu")
+(net 4)
+	)
+	(segment
 (start 158.1000 108.8000)
 (end 158.1000 108.6000)
@@
 	)
 	(segment
+(start 158.0000 101.0000)
+(end 159.8000 101.0000)
+(width 0.2)
+(layer "B.Cu")
+(net 4)
+	)
+	(segment
+(start 158.0000 87.0000)
+(end 158.0000 85.5000)
+(width 0.2)
+(layer "B.Cu")
+(net 4)
+	)
+	(segment
 (start 142.2000 91.9000)
 (end 141.6000 92.5000)
@@
 	)
 	(via
-(at 145.800 86.200)
-(size 0.6)
-(drill 0.3)
-(layers "F.Cu" "B.Cu")
-(net 4)
-	)
-	(via
-(at 145.800 88.600)
-(size 0.6)
-(drill 0.3)
-(layers "F.Cu" "B.Cu")
-(net 4)
-	)
-	(via
-(at 145.800 91.000)
-(size 0.6)
-(drill 0.3)
-(layers "F.Cu" "B.Cu")
-(net 4)
-	)
-	(via
-(at 145.800 93.400)
-(size 0.6)
-(drill 0.3)
-(layers "F.Cu" "B.Cu")
-(net 4)
-	)
-	(via
-(at 145.800 95.800)
-(size 0.6)
-(drill 0.3)
-(layers "F.Cu" "B.Cu")
-(net 4)
-	)
-	(via
-(at 145.800 98.200)
-(size 0.6)
-(drill 0.3)
-(layers "F.Cu" "B.Cu")
-(net 4)
-	)
-	(via
-(at 145.800 100.600)
-(size 0.6)
-(drill 0.3)
-(layers "F.Cu" "B.Cu")
-(net 4)
-	)
-	(via
 (at 145.800 110.200)
 (size 0.6)
@@
 	)
 	(via
-(at 148.200 86.200)
-(size 0.6)
-(drill 0.3)
-(layers "F.Cu" "B.Cu")
-(net 4)
-	)
-	(via
-(at 148.200 88.600)
-(size 0.6)
-(drill 0.3)
-(layers "F.Cu" "B.Cu")
-(net 4)
-	)
-	(via
 (at 148.200 119.800)
 (size 0.6)
@@
 	)
 	(via
-(at 150.600 86.200)
-(size 0.6)
-(drill 0.3)
-(layers "F.Cu" "B.Cu")
-(net 4)
-	)
-	(via
-(at 150.600 88.600)
-(size 0.6)
-(drill 0.3)
-(layers "F.Cu" "B.Cu")
-(net 4)
-	)
-	(via
-(at 150.600 100.600)
-(size 0.6)
-(drill 0.3)
-(layers "F.Cu" "B.Cu")
-(net 4)
-	)
-	(via
 (at 150.600 119.800)
 (size 0.6)
@@
 	)
 	(via
-(at 153.000 86.200)
-(size 0.6)
-(drill 0.3)
-(layers "F.Cu" "B.Cu")
-(net 4)
-	)
-	(via
-(at 153.000 88.600)
-(size 0.6)
-(drill 0.3)
-(layers "F.Cu" "B.Cu")
-(net 4)
-	)
-	(via
-(at 153.000 91.000)
-(size 0.6)
-(drill 0.3)
-(layers "F.Cu" "B.Cu")
-(net 4)
-	)
-	(via
-(at 153.000 98.200)
-(size 0.6)
-(drill 0.3)
-(layers "F.Cu" "B.Cu")
-(net 4)
-	)
-	(via
 (at 153.000 105.400)
 (size 0.6)
@@
 	)
 	(via
-(at 155.400 86.200)
-(size 0.6)
-(drill 0.3)
-(layers "F.Cu" "B.Cu")
-(net 4)
-	)
-	(via
-(at 155.400 88.600)
-(size 0.6)
-(drill 0.3)
-(layers "F.Cu" "B.Cu")
-(net 4)
-	)
-	(via
-(at 155.400 95.800)
-(size 0.6)
-(drill 0.3)
-(layers "F.Cu" "B.Cu")
-(net 4)
-	)
-	(via
-(at 155.400 100.600)
-(size 0.6)
-(drill 0.3)
-(layers "F.Cu" "B.Cu")
-(net 4)
-	)
-	(via
 (at 155.400 105.400)
 (size 0.6)
@@
 (size 0.6)
 (drill 0.3)
-(layers "F.Cu" "B.Cu")
-(net 4)
-	)
-	(via
-(at 160.200 110.200)
-(size 0.6)
-(drill 0.3)
