File: hardware/pcb/v2/kaelix.kicad_pcb (KiCad board)
At the start: 2 copper layers, 61 x 51 mm, 35 parts, among them J1 LiPo 3,7V, J2 UART/BOOT, Q1 SI2301CDS, Q2 BC847B, Q3 SI2301CDS, U1 ESP32-S3-WROOM-1U-N16R8, U2 MPU-6050, U3 Ai-Thinker Ra-02 (SX1278), U4 HT7333

Commit message: fix(router): não conta plano sob o corpo de peça de passo fino
A grade do roteador via células de plano de terra na faixa entre as
fileiras de pads de um QFN de 0,5 mm e tratava a região como caminho. O
preenchimento do KiCad, com espessura mínima e folga exatas, deixa ali só
retalhos, e o escape seguinte ou uma pista de sinal os fecha em ilha. Na
v3 o escape de GND do U2.1 terminou numa dessas ilhas sob o MPU6050: o
roteador deu o pad por ligado e o DRC acusou um grupo de terra solto.

Agora, sob o corpo de peça de passo fino e na face dela, o plano não conta
como caminho. Atravessar com pista continua possível; só deixa de valer
contar com plano ali. A regra fica no modelo do plano (_gnd_ok), e não em
cada ponto de chegada, porque o escape inicial e a verificação final de
terra usam o mesmo modelo.

O roteamento da v1 e da v2 muda — costura 92 -> 71 e 261 -> 234, porque a
região deixou de oferecer plano dos dois lados — sem tocar em circuito nem
em placement. As duas seguem com ERC e DRC limpos e zero itens soltos.
Routing:
- net GND: track 3.26 -> 9.16 mm, vias 262 -> 236
Changed lines of the file:
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@@
 	)
 	(segment
+(start 134.1000 110.6000)
+(end 128.2000 110.6000)
+(width 0.2)
+(layer "B.Cu")
+(net 4)
+	)
+	(segment
 (start 148.1000 86.7000)
 (end 147.9000 86.5000)
@@
 (net 4)
 	)
+	(via
+(at 145.8000 103.6000)
+(size 0.6)
+(drill 0.3)
+(layers "F.Cu" "B.Cu")
+(net 4)
+	)
 	(zone
 (net 4)
@@
 	)
 	(via
-(at 131.500 110.300)
-(size 0.6)
-(drill 0.3)
-(layers "F.Cu" "B.Cu")
-(net 4)
-	)
-	(via
-(at 131.500 112.700)
-(size 0.6)
-(drill 0.3)
-(layers "F.Cu" "B.Cu")
-(net 4)
-	)
-	(via
-(at 131.500 115.100)
-(size 0.6)
-(drill 0.3)
-(layers "F.Cu" "B.Cu")
-(net 4)
-	)
-	(via
-(at 131.500 117.500)
-(size 0.6)
-(drill 0.3)
-(layers "F.Cu" "B.Cu")
-(net 4)
-	)
-	(via
-(at 131.500 119.900)
-(size 0.6)
-(drill 0.3)
-(layers "F.Cu" "B.Cu")
-(net 4)
-	)
-	(via
 (at 133.900 76.700)
 (size 0.6)
@@
 	)
 	(via
-(at 133.900 105.500)
-(size 0.6)
-(drill 0.3)
-(layers "F.Cu" "B.Cu")
-(net 4)
-	)
-	(via
-(at 133.900 115.100)
-(size 0.6)
-(drill 0.3)
-(layers "F.Cu" "B.Cu")
-(net 4)
-	)
-	(via
-(at 133.900 117.500)
-(size 0.6)
-(drill 0.3)
-(layers "F.Cu" "B.Cu")
-(net 4)
-	)
-	(via
 (at 136.300 76.700)
 (size 0.6)
@@
 	)
 	(via
-(at 136.300 107.900)
-(size 0.6)
-(drill 0.3)
-(layers "F.Cu" "B.Cu")
-(net 4)
-	)
-	(via
-(at 136.300 115.100)
-(size 0.6)
-(drill 0.3)
-(layers "F.Cu" "B.Cu")
-(net 4)
-	)
-	(via
-(at 136.300 119.900)
-(size 0.6)
-(drill 0.3)
-(layers "F.Cu" "B.Cu")
-(net 4)
-	)
-	(via
 (at 138.700 76.700)
 (size 0.6)
@@
 	)
 	(via
-(at 138.700 105.500)
-(size 0.6)
-(drill 0.3)
-(layers "F.Cu" "B.Cu")
-(net 4)
-	)
-	(via
-(at 138.700 107.900)
-(size 0.6)
-(drill 0.3)
-(layers "F.Cu" "B.Cu")
-(net 4)
-	)
-	(via
-(at 138.700 110.300)
-(size 0.6)
-(drill 0.3)
-(layers "F.Cu" "B.Cu")
-(net 4)
-	)
-	(via
-(at 138.700 112.700)
-(size 0.6)
-(drill 0.3)
-(layers "F.Cu" "B.Cu")
-(net 4)
-	)
-	(via
-(at 138.700 117.500)
-(size 0.6)
-(drill 0.3)
-(layers "F.Cu" "B.Cu")
-(net 4)
-	)
-	(via
-(at 138.700 119.900)
-(size 0.6)
-(drill 0.3)
-(layers "F.Cu" "B.Cu")
-(net 4)
-	)
-	(via
 (at 141.100 76.700)
 (size 0.6)
@@
 	)
 	(via
-(at 141.100 105.500)
-(size 0.6)
-(drill 0.3)
-(layers "F.Cu" "B.Cu")
-(net 4)
-	)
-	(via
-(at 141.100 107.900)
-(size 0.6)
-(drill 0.3)
-(layers "F.Cu" "B.Cu")
-(net 4)
-	)
-	(via
-(at 141.100 110.300)
-(size 0.6)
-(drill 0.3)
-(layers "F.Cu" "B.Cu")
-(net 4)
-	)
-	(via
-(at 141.100 115.100)
-(size 0.6)
-(drill 0.3)
-(layers "F.Cu" "B.Cu")
-(net 4)
-	)
-	(via
-(at 141.100 117.500)
-(size 0.6)
-(drill 0.3)
-(layers "F.Cu" "B.Cu")
-(net 4)
-	)
-	(via
 (at 143.500 76.700)
 (size 0.6)
@@
 (size 0.6)
 (drill 0.3)
-(layers "F.Cu" "B.Cu")
-(net 4)
-	)
-	(via
-(at 143.500 105.500)
-(size 0.6)
-(drill 0.3)
-(layers "F.Cu" "B.Cu")
-(net 4)
-	)
-	(via
-(at 143.500 107.900)
-(size 0.6)
-(drill 0.3)
-(layers "F.Cu" "B.Cu")
-(net 4)
-	)
-	(via
-(at 143.500 112.700)
-(size 0.6)
-(drill 0.3)
-(layers "F.Cu" "B.Cu")
-(net 4)
-	)
-	(via
-(at 143.500 115.100)
-(size 0.6)
-(drill 0.3)
-(layers "F.Cu" "B.Cu")
-(net 4)
-	)
-	(via
-(at 143.500 117.500)
-(size 0.6)
-(drill 0.3)
